Commit message: adding some simple c serial stuff for alex, he needs to solve the crimes with the cameras as crimes are being commited with the camera crimes

File: Test_Ground/gazebo_test/object.urdf (robot description, URDF)
Before this commit: robot simple_box, 1 links, 0 joints
Links:
- link my_box: geometry collision box size=1 1 2; visual box size=0.1 2 0.1
